File: usbc_power_supply_2.kicad_pcb (KiCad board)
At the start: 2 copper layers, 25 x 25 mm, 22 parts, among them J1 USB4125-GF-A-0190, J2 B2B-PH-K-SLFSN, J3 B2B-PH-K-SLFSN, Q1 DMG3415UFY4Q-7, U1 MBR0540T3G, U2 MCP73833-AMI/MF

Commit message: updates mounting holes with pads, optional 1A shottkyx
Parts:
- H1, H2: footprint MountingHole:MountingHole_2.2mm_M2 -> MountingHole:MountingHole_2.2mm_M2_Pad
- U1: value MBR0540T3G -> MBR0540T3G (500mA) or PMEG3010EGW (1A)
Changed lines of the file:
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@@
         (effects (font (size 1 1) (thickness 0.15)))
     )
-    (fp_text value "MBR0540T3G" (at 1.1364 -3.34 90 unlocked) (layer "F.Fab") hide
+    (fp_text value "MBR0540T3G (500mA) or  PMEG3010EGW  (1A)" (at 1.1364 -3.34 90 unlocked) (layer "F.Fab") hide
         (effects (font (size 1 1) (thickness 0.15)))
     )
@@
     (pad "13" thru_hole circle (at -1.570007 3.800006 180) (size 0.762 0.762) (drill 0.508) (layers "*.Cu" "*.Mask"))
   )
-  (footprint "MountingHole:MountingHole_2.2mm_M2" (layer "F.Cu")
+  (footprint "MountingHole:MountingHole_2.2mm_M2_Pad" (layer "F.Cu")
     (at 103.25 103.25)
-    (descr "Mounting Hole 2.2mm, no annular, M2")
-    (tags "mounting hole 2.2mm no annular m2")
+    (descr "Mounting Hole 2.2mm, M2")
+    (tags "mounting hole 2.2mm m2")
     (property "Sheetfile" "usbc_power_supply_2.kicad_sch")
     (property "Sheetname" "")
@@
         (effects (font (size 1 1) (thickness 0.15)))
     )
-    (fp_text value "Mount" (at 0 3.2) (layer "F.Fab") hide
+    (fp_text value "Mount" (at 0 3.2) (layer "F.Fab")
         (effects (font (size 1 1) (thickness 0.15)))
     )
@@
     (fp_circle (center 0 0) (end 2.45 0)
       (stroke (width 0.05) (type solid)) (fill none) (layer "F.CrtYd"))
-    (pad "" np_thru_hole circle (at 0 0) (size 2.2 2.2) (drill 2.2) (layers "*.Cu" "*.Mask"))
+    (pad "1" thru_hole circle (at 0 0) (size 4.4 4.4) (drill 2.2) (layers "*.Cu" "*.Mask")
+      (net 2 "GND") (pinfunction "1") (pintype "input"))
   )
   (footprint "AMU-Resistors:ERJ6G_PAN" (layer "F.Cu")
@@
       (net 3 "VBUS") (pinfunction "A") (pintype "passive") (thermal_bridge_angle 45))
   )
-  (footprint "MountingHole:MountingHole_2.2mm_M2" (layer "F.Cu")
+  (footprint "MountingHole:MountingHole_2.2mm_M2_Pad" (layer "F.Cu")
     (at 121.75 103.25)
-    (descr "Mounting Hole 2.2mm, no annular, M2")
-    (tags "mounting hole 2.2mm no annular m2")
+    (descr "Mounting Hole 2.2mm, M2")
+    (tags "mounting hole 2.2mm m2")
     (property "Sheetfile" "usbc_power_supply_2.kicad_sch")
     (property "Sheetname" "")
@@
         (effects (font (size 1 1) (thickness 0.15)))
     )
-    (fp_text value "Mount" (at 0 3.2) (layer "F.Fab") hide
+    (fp_text value "Mount" (at 0 3.2) (layer "F.Fab")
         (effects (font (size 1 1) (thickness 0.15)))
     )
@@
     (fp_circle (center 0 0) (end 2.45 0)
       (stroke (width 0.05) (type solid)) (fill none) (layer "F.CrtYd"))
-    (pad "" np_thru_hole circle (at 0 0) (size 2.2 2.2) (drill 2.2) (layers "*.Cu" "*.Mask"))
+    (pad "1" thru_hole circle (at 0 0) (size 4.4 4.4) (drill 2.2) (layers "*.Cu" "*.Mask")
+      (net 2 "GND") (pinfunction "1") (pintype "input"))
   )
   (footprint "AMU-Capacitors:C0805" (layer "F.Cu")
@@
   )
   (dimension (type aligned) (layer "User.1")
-    (pts (xy 100 125) (xy 109.3 125))
-    (height 5.4)
-    (gr_text "9.3000 mm" (at 104.65 129.25) (layer "User.1")
-      (effects (font (size 1 1) (thickness 0.15)))
-    )
-    (format (prefix "") (suffix "") (units 3) (units_format 1) (precision 4))
-    (style (thickness 0.15) (arrow_length 1.27) (text_position_mode 0) (extension_height 0.58642) (extension_offset 0.5) keep_text_aligned)
-  )
-  (dimension (type aligned) (layer "User.1")
     (pts (xy 125 100) (xy 121.75 100))
     (height 3.45)
@@
   )
   (dimension (type aligned) (layer "User.1")
-    (pts (xy 123.95 123.925) (xy 123.95 125.05))
-    (height -6.78)
-    (gr_text "1.1250 mm" (at 129.58 124.4875 90) (layer "User.1")
+    (pts (xy 100 125) (xy 125 125))
+    (height 7.19)
+    (gr_text "25.0000 mm" (at 112.5 131.04) (layer "User.1")
       (effects (font (size 1 1) (thickness 0.15)))
     )
@@
   )
   (dimension (type aligned) (layer "User.1")
-    (pts (xy 123.95 123.925) (xy 125.05 123.93))
-    (height 3.688591)
-    (gr_text "1.1000 mm" (at 124.488461 126.466065 359.7395664) (layer "User.1")
+    (pts (xy 100 100) (xy 100 125))
+    (height 10.59)
+    (gr_text "25.0000 mm" (at 88.26 112.5 90) (layer "User.1")
       (effects (font (size 1 1) (thickness 0.15)))
     )
